Commit message: Added v2 collision mesh

File: v2/models/urdf/orcahand_left.urdf (robot description, URDF)
Before this commit: robot orcahand_left, 19 links, 18 joints
Links:
- link ForeArmStructure-Model_e18f2368: geometry collision mesh filename=package://orcahand_description/v2/models/assets/left/collis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 scale=0.001 0.001 0.001; visual mesh filename=package://orcahand_description/v2/models/assets/left/ForeAr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 scale=0.001 0.001 0.001
- link I-AP-L_57ce92f7: geometry collision mesh filename=package://orcahand_description/v2/models/assets/left/collis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 scale=0.001 0.001 0.001; visual mesh filename=package://orcahand_description/v2/models/assets/left/I-AP-L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 scale=0.001 0.001 0.001
- link I-FingerTipAssembly_ed91b18a: geometry collision mesh filename=package://orcahand_description/v2/models/assets/left/collis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 scale=0.001 0.001 0.001; collision mesh filename=package://orcahand_description/v2/models/assets/left/collis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 scale=0.001 0.001 0.001
- link I-PP_3df4f91d: geometry collision mesh filename=package://orcahand_description/v2/models/assets/left/collis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 scale=0.001 0.001 0.001; collision mesh filename=package://orcahand_description/v2/models/assets/left/collis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 scale=0.001 0.001 0.001
- link L-Carpals_719fff8c: geometry collision mesh filename=package://orcahand_description/v2/models/assets/left/collis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 scale=0.001 0.001 0.001; collision mesh filename=package://orcahand_description/v2/models/assets/left/collis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 scale=0.001 0.001 0.001
- link L-T-AP_58680c44: geometry collision mesh filename=package://orcahand_description/v2/models/assets/left/collis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 scale=0.001 0.001 0.001; visual mesh filename=package://orcahand_description/v2/models/assets/left/L-T-AP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 scale=0.001 0.001 0.001
- link M-AP_6ec59111: geometry collision mesh filename=package://orcahand_description/v2/models/assets/left/collis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 scale=0.001 0.001 0.001; visual mesh filename=package://orcahand_description/v2/models/assets/left/M-AP.s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 scale=0.001 0.001 0.001
- link M-AP_e04a96f2: geometry collision mesh filename=package://orcahand_description/v2/models/assets/left/collis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 scale=0.001 0.001 0.001; visual mesh filename=package://orcahand_description/v2/models/assets/left/M-AP.s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 scale=0.001 0.001 0.001
- link M-FingerTipAssembly_34afb748: geometry collision mesh filename=package://orcahand_description/v2/models/assets/left/collis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 scale=0.001 0.001 0.001; collision mesh filename=package://orcahand_description/v2/models/assets/left/collis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 scale=0.001 0.001 0.001
- link M-FingerTipAssembly_424a8e75: geometry collision mesh filename=package://orcahand_description/v2/models/assets/left/collis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 scale=0.001 0.001 0.001; collision mesh filename=package://orcahand_description/v2/models/assets/left/collis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 scale=0.001 0.001 0.001
- link M-PP_08efa608: geometry collision mesh filename=package://orcahand_description/v2/models/assets/left/collis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 scale=0.001 0.001 0.001; collision mesh filename=package://orcahand_description/v2/models/assets/left/collis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 scale=0.001 0.001 0.001
- link M-PP_8660a1eb: geometry collision mesh filename=package://orcahand_description/v2/models/assets/left/collis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 scale=0.001 0.001 0.001; collision mesh filename=package://orcahand_description/v2/models/assets/left/collis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 scale=0.001 0.001 0.001
- link P-AP_f5e42b61: geometry collision mesh filename=package://orcahand_description/v2/models/assets/left/collis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 scale=0.001 0.001 0.001; visual mesh filename=package://orcahand_description/v2/models/assets/left/P-AP.s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 scale=0.001 0.001 0.001
- link P-FingerTipAssembly_cd219176: geometry collision mesh filename=package://orcahand_description/v2/models/assets/left/collis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 scale=0.001 0.001 0.001; collision mesh filename=package://orcahand_description/v2/models/assets/left/collis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 scale=0.001 0.001 0.001
- link P-PP_1d411b9b: geometry collision mesh filename=package://orcahand_description/v2/models/assets/left/collis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 scale=0.001 0.001 0.001; collision mesh filename=package://orcahand_description/v2/models/assets/left/collis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 scale=0.001 0.001 0.001
- link T-DP_307db3cc: geometry collision mesh filename=package://orcahand_description/v2/models/assets/left/collis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 scale=0.001 0.001 0.001; collision mesh filename=package://orcahand_description/v2/models/assets/left/collis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 scale=0.001 0.001 0.001
- link T-PP_ef067304: geometry collision mesh filename=package://orcahand_description/v2/models/assets/left/collis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 scale=0.001 0.001 0.001; collision mesh filename=package://orcahand_description/v2/models/assets/left/collis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 scale=0.001 0.001 0.001
- link T-TP-L_92b8100b: geometry collision mesh filename=package://orcahand_description/v2/models/assets/left/collis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 scale=0.001 0.001 0.001; visual mesh filename=package://orcahand_description/v2/models/assets/left/T-TP-L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 scale=0.001 0.001 0.001
- link TopTower-Model_4a80d30e: geometry collision mesh filename=package://orcahand_description/v2/models/assets/left/collis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 scale=0.001 0.001 0.001; visual mesh filename=package://orcahand_description/v2/models/assets/left/TopTow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 scale=0.001 0.001 0.001

File: v2/models/urdf/orcahand_right.urdf (robot description, URDF)
Before this commit: robot orcahand_right, 19 links, 18 joints
Links:
- link ForeArmStructure-Model_e18f2368: geometry collision mesh filename=package://orcahand_description/v2/models/assets/right/colli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 scale=0.001 0.001 0.001; visual mesh filename=package://orcahand_description/v2/models/assets/right/ForeA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 scale=0.001 0.001 0.001
- link I-AP-R_d95d02d1: geometry collision mesh filename=package://orcahand_description/v2/models/assets/right/colli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 scale=0.001 0.001 0.001; visual mesh filename=package://orcahand_description/v2/models/assets/right/I-AP-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 scale=0.001 0.001 0.001
- link I-FingerTipAssembly_ec49c16c: geometry collision mesh filename=package://orcahand_description/v2/models/assets/right/colli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 scale=0.001 0.001 0.001; collision mesh filename=package://orcahand_description/v2/models/assets/right/colli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 scale=0.001 0.001 0.001
- link I-PP_bacbd481: geometry collision mesh filename=package://orcahand_description/v2/models/assets/right/colli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 scale=0.001 0.001 0.001; collision mesh filename=package://orcahand_description/v2/models/assets/right/colli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 scale=0.001 0.001 0.001
- link M-AP_6ec59111: geometry collision mesh filename=package://orcahand_description/v2/models/assets/right/colli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 scale=0.001 0.001 0.001; visual mesh filename=package://orcahand_description/v2/models/assets/right/M-AP.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 scale=0.001 0.001 0.001
- link M-AP_e04a96f2: geometry collision mesh filename=package://orcahand_description/v2/models/assets/right/colli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 scale=0.001 0.001 0.001; visual mesh filename=package://orcahand_description/v2/models/assets/right/M-AP.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 scale=0.001 0.001 0.001
- link M-FingerTipAssembly_34afb748: geometry collision mesh filename=package://orcahand_description/v2/models/assets/right/colli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 scale=0.001 0.001 0.001; collision mesh filename=package://orcahand_description/v2/models/assets/right/colli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 scale=0.001 0.001 0.001
- link M-FingerTipAssembly_424a8e75: geometry collision mesh filename=package://orcahand_description/v2/models/assets/right/colli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 scale=0.001 0.001 0.001; collision mesh filename=package://orcahand_description/v2/models/assets/right/colli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 scale=0.001 0.001 0.001
- link M-PP_08efa608: geometry collision mesh filename=package://orcahand_description/v2/models/assets/right/colli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 scale=0.001 0.001 0.001; collision mesh filename=package://orcahand_description/v2/models/assets/right/colli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 scale=0.001 0.001 0.001
- link M-PP_8660a1eb: geometry collision mesh filename=package://orcahand_description/v2/models/assets/right/colli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 scale=0.001 0.001 0.001; collision mesh filename=package://orcahand_description/v2/models/assets/right/colli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 scale=0.001 0.001 0.001
- link P-AP_f5e42b61: geometry collision mesh filename=package://orcahand_description/v2/models/assets/right/colli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 scale=0.001 0.001 0.001; visual mesh filename=package://orcahand_description/v2/models/assets/right/P-AP.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 scale=0.001 0.001 0.001
- link P-FingerTipAssembly_cd219176: geometry collision mesh filename=package://orcahand_description/v2/models/assets/right/colli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 scale=0.001 0.001 0.001; collision mesh filename=package://orcahand_description/v2/models/assets/right/colli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 scale=0.001 0.001 0.001
- link P-PP_1d411b9b: geometry collision mesh filename=package://orcahand_description/v2/models/assets/right/colli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 scale=0.001 0.001 0.001; collision mesh filename=package://orcahand_description/v2/models/assets/right/colli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 scale=0.001 0.001 0.001
- link R-Carpals_8d1f1041: geometry collision mesh filename=package://orcahand_description/v2/models/assets/right/colli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 scale=0.001 0.001 0.001; collision mesh filename=package://orcahand_description/v2/models/assets/right/colli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 scale=0.001 0.001 0.001
- link R-T-AP_a9723101: geometry collision mesh filename=package://orcahand_description/v2/models/assets/right/colli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 scale=0.001 0.001 0.001; visual mesh filename=package://orcahand_description/v2/models/assets/right/R-T-A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 scale=0.001 0.001 0.001
- link T-DP_b7429e50: geometry collision mesh filename=package://orcahand_description/v2/models/assets/right/colli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 scale=0.001 0.001 0.001; collision mesh filename=package://orcahand_description/v2/models/assets/right/colli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 scale=0.001 0.001 0.001
- link T-PP_68395e98: geometry collision mesh filename=package://orcahand_description/v2/models/assets/right/colli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 scale=0.001 0.001 0.001; collision mesh filename=package://orcahand_description/v2/models/assets/right/colli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 scale=0.001 0.001 0.001
- link T-TP-R_1c2b802d: geometry collision mesh filename=package://orcahand_description/v2/models/assets/right/colli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 scale=0.001 0.001 0.001; visual mesh filename=package://orcahand_description/v2/models/assets/right/T-TP-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 scale=0.001 0.001 0.001
- link TopTower-Model_4a80d30e: geometry collision mesh filename=package://orcahand_description/v2/models/assets/right/colli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 scale=0.001 0.001 0.001; visual mesh filename=package://orcahand_description/v2/models/assets/right/TopTo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 scale=0.001 0.001 0.001
