Commit message: Rename v2 joints/links/bodies from Fusion hashes to semantic names
Port of upstream orcahand/orcahand_description 0818eae (branch
fb/split-mjcf-scene-positioning), which this fork's main lacked. Joints are
now {side}_{orca_core joint id} (right_index_mcp, left_thumb_dip) in both URDF
and MJCF, as orca_core's tools/extract_urdf_kinematics.py requires, and the
thumb DIP is no longer misnamed t-pip. Links and MJCF bodies use semantic part
names ({side}_carpals, {side}_ring_pp); the MJCF root wrapper body is
{side}_base, and {side}_tower is now the TopTower body. Mesh files, mesh asset
names and the collision classes keep their names.

Applied as a single-pass old->new name map derived from 0818eae's own
before/after files, so the renamed files carry exactly upstream's name set plus
this fork's collision meshes. mirror_left_from_right.py loses its hash LINK_MAP
and additionally generates orcahand_left.mjcf; README gains upstream's naming
section.

Pure rename: the compiled MuJoCo models are numerically identical before and
after. Breaking for users of the old MJCF names (right_i-mcp -> right_index_mcp,
right_t-pip -> right_thumb_dip, root body right_tower -> right_base).

Co-Authored-By: Claude Opus 5.5 <noreply@anthropic.com>

File: v2/models/urdf/orcahand_right.urdf (robot description, URDF)
Before this commit: robot orcahand_right, 19 links, 18 joints
Links:
- removed link ForeArmStructure-Model_e18f2368
- removed link I-AP-R_d95d02d1
- removed link I-FingerTipAssembly_ec49c16c
- removed link I-PP_bacbd481
- removed link M-AP_6ec59111
- removed link M-AP_e04a96f2
- removed link M-FingerTipAssembly_34afb748
- removed link M-FingerTipAssembly_424a8e75
- removed link M-PP_08efa608
- removed link M-PP_8660a1eb
- removed link P-AP_f5e42b61
- removed link P-FingerTipAssembly_cd219176
- removed link P-PP_1d411b9b
- removed link R-Carpals_8d1f1041
- removed link R-T-AP_a9723101
- removed link T-DP_b7429e50
- removed link T-PP_68395e98
- removed link T-TP-R_1c2b802d
- removed link TopTower-Model_4a80d30e
- added link right_carpals, mass 0.13538810897856451; collision mesh filename=package://orcahand_description/v2/models/assets/right/colli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 scale=0.001 0.001 0.001; collision mesh filename=package://orcahand_description/v2/models/assets/right/colli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 scale=0.001 0.001 0.001
- added link right_forearm, mass 7.422534035794272; collision mesh filename=package://orcahand_description/v2/models/assets/right/colli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 scale=0.001 0.001 0.001; visual mesh filename=package://orcahand_description/v2/models/assets/right/ForeA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 scale=0.001 0.001 0.001
- added link right_index_ap, mass 0.004590288233037025; collision mesh filename=package://orcahand_description/v2/models/assets/right/colli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 scale=0.001 0.001 0.001; visual mesh filename=package://orcahand_description/v2/models/assets/right/I-AP-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 scale=0.001 0.001 0.001
- added link right_index_fingertip_assembly, mass 0.04675178908397048; collision mesh filename=package://orcahand_description/v2/models/assets/right/colli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 scale=0.001 0.001 0.001; collision mesh filename=package://orcahand_description/v2/models/assets/right/colli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 scale=0.001 0.001 0.001
- added link right_index_pp, mass 0.011373207304546197; collision mesh filename=package://orcahand_description/v2/models/assets/right/colli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 scale=0.001 0.001 0.001; collision mesh filename=package://orcahand_description/v2/models/assets/right/colli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 scale=0.001 0.001 0.001
- added link right_middle_ap, mass 0.004923565158859135; collision mesh filename=package://orcahand_description/v2/models/assets/right/colli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 scale=0.001 0.001 0.001; visual mesh filename=package://orcahand_description/v2/models/assets/right/M-AP.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 scale=0.001 0.001 0.001
- added link right_middle_fingertip_assembly, mass 0.04673701376980013; collision mesh filename=package://orcahand_description/v2/models/assets/right/colli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 scale=0.001 0.001 0.001; collision mesh filename=package://orcahand_description/v2/models/assets/right/colli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 scale=0.001 0.001 0.001
- added link right_middle_pp, mass 0.012733573971304512; collision mesh filename=package://orcahand_description/v2/models/assets/right/colli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 scale=0.001 0.001 0.001; collision mesh filename=package://orcahand_description/v2/models/assets/right/colli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 scale=0.001 0.001 0.001
- added link right_pinky_ap, mass 0.004135862855401387; collision mesh filename=package://orcahand_description/v2/models/assets/right/colli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 scale=0.001 0.001 0.001; visual mesh filename=package://orcahand_description/v2/models/assets/right/P-AP.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 scale=0.001 0.001 0.001
- added link right_pinky_fingertip_assembly, mass 0.033190557637887204; collision mesh filename=package://orcahand_description/v2/models/assets/right/colli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 scale=0.001 0.001 0.001; collision mesh filename=package://orcahand_description/v2/models/assets/right/colli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 scale=0.001 0.001 0.001
- added link right_pinky_pp, mass 0.008117379921259958; collision mesh filename=package://orcahand_description/v2/models/assets/right/colli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 scale=0.001 0.001 0.001; collision mesh filename=package://orcahand_description/v2/models/assets/right/colli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 scale=0.001 0.001 0.001
- added link right_ring_ap, mass 0.004923565158859135; collision mesh filename=package://orcahand_description/v2/models/assets/right/colli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 scale=0.001 0.001 0.001; visual mesh filename=package://orcahand_description/v2/models/assets/right/M-AP.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 scale=0.001 0.001 0.001
- added link right_ring_fingertip_assembly, mass 0.04673701376980013; collision mesh filename=package://orcahand_description/v2/models/assets/right/colli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 scale=0.001 0.001 0.001; collision mesh filename=package://orcahand_description/v2/models/assets/right/colli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 scale=0.001 0.001 0.001
- added link right_ring_pp, mass 0.012733573971304512; collision mesh filename=package://orcahand_description/v2/models/assets/right/colli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 scale=0.001 0.001 0.001; collision mesh filename=package://orcahand_description/v2/models/assets/right/colli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 scale=0.001 0.001 0.001
- added link right_thumb_ap, mass 0.007004136465100992; collision mesh filename=package://orcahand_description/v2/models/assets/right/colli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 scale=0.001 0.001 0.001; visual mesh filename=package://orcahand_description/v2/models/assets/right/R-T-A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 scale=0.001 0.001 0.001
- added link right_thumb_dp, mass 0.00815768733004441; collision mesh filename=package://orcahand_description/v2/models/assets/right/colli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 scale=0.001 0.001 0.001; collision mesh filename=package://orcahand_description/v2/models/assets/right/colli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 scale=0.001 0.001 0.001
- added link right_thumb_pp, mass 0.010490827160908196; collision mesh filename=package://orcahand_description/v2/models/assets/right/colli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 scale=0.001 0.001 0.001; collision mesh filename=package://orcahand_description/v2/models/assets/right/colli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 scale=0.001 0.001 0.001
- added link right_thumb_tp, mass 0.00797873207561227; collision mesh filename=package://orcahand_description/v2/models/assets/right/colli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 scale=0.001 0.001 0.001; visual mesh filename=package://orcahand_description/v2/models/assets/right/T-TP-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 scale=0.001 0.001 0.001
- added link right_tower, mass 0.18565193224536478; collision mesh filename=package://orcahand_description/v2/models/assets/right/colli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 scale=0.001 0.001 0.001; visual mesh filename=package://orcahand_description/v2/models/assets/right/TopTo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 scale=0.001 0.001 0.001
Joints:
- removed joint I-AP-R_d95d02d1_to_R-Carpals_8d1f1041
- removed joint I-FingerTipAssembly_ec49c16c_to_I-PP_bacbd481
- removed joint I-PP_bacbd481_to_I-AP-R_d95d02d1
- removed joint M-AP_6ec59111_to_R-Carpals_8d1f1041
- removed joint M-AP_e04a96f2_to_R-Carpals_8d1f1041
- removed joint M-FingerTipAssembly_34afb748_to_M-PP_08efa608
- removed joint M-FingerTipAssembly_424a8e75_to_M-PP_8660a1eb
- removed joint M-PP_08efa608_to_M-AP_e04a96f2
- removed joint M-PP_8660a1eb_to_M-AP_6ec59111
- removed joint P-AP_f5e42b61_to_R-Carpals_8d1f1041
- removed joint P-FingerTipAssembly_cd219176_to_P-PP_1d411b9b
- removed joint P-PP_1d411b9b_to_P-AP_f5e42b61
- removed joint R-Carpals_8d1f1041_to_TopTower-Model_4a80d30e
- removed joint R-T-AP_a9723101_to_T-TP-R_1c2b802d
- removed joint T-DP_b7429e50_to_T-PP_68395e98
- removed joint T-PP_68395e98_to_R-T-AP_a9723101
- removed joint T-TP-R_1c2b802d_to_R-Carpals_8d1f1041
- removed joint TopTower-Model_4a80d30e_to_ForeArmStructure-Model_e18f2368
- added joint right_index_abd: type revolute, parent right_carpals, child right_index_ap, origin xyz=-0.027240979039914386 -0.002206966804174762 0.06940680269673646 rpy=1.6538568135338134 1.3873496487488786 -0.0042742186040372054, axis -8.326672684688674e-17 3.3306690738754696e-16 0.9999999999999991, limit lower=-0.4363323129985824 upper=0.5235987755982988 effort=100 velocity=100
- added joint right_index_mcp: type revolute, parent right_index_ap, child right_index_pp, origin xyz=-0.01915096815087666 -4.499288227880137e-18 -0.0009999999999971549 rpy=-2.9439233600320843e-16 -1.570796326794891 0.0, axis 5.828670879282072e-15 -1.0000000000000036 1.1102230246251565e-16, limit lower=-0.4363323129985824 upper=1.7453292519943295 effort=100 velocity=100
- added joint right_index_pip: type revolute, parent right_index_pp, child right_index_fingertip_assembly, origin xyz=0.0015000000000000417 -7.819255613844171e-18 0.037000000000000026 rpy=3.3306690738754617e-16 0.0 6.77236045021344e-15, axis -3.608224830031759e-15 -0.999999999999996 2.7755575615628914e-16, limit lower=-0.2617993877991494 upper=1.8675022996339325 effort=100 velocity=100
- added joint right_middle_abd: type revolute, parent right_carpals, child right_middle_ap, origin xyz=-0.005706333727246699 -0.004023404072025678 0.07850189342716887 rpy=1.5707963267946425 1.5681783329169052 -2.544631172440859e-13, axis 1.1102230246251565e-15 -2.220446049250313e-16 0.9999999999999971, limit lower=-0.47123889803846897 upper=0.47123889803846897 effort=100 velocity=100
- added joint right_middle_mcp: type revolute, parent right_middle_ap, child right_middle_pp, origin xyz=-0.019866967942905277 -1.8423293703642938e-17 -0.0009999999999957202 rpy=0.0 -1.5707963267948903 0.0, axis 6.050715484207103e-15 -1.0000000000000058 -1.1102230246251565e-16, limit lower=-0.4363323129985824 upper=1.7453292519943295 effort=100 velocity=100
- added joint right_middle_pip: type revolute, parent right_middle_pp, child right_middle_fingertip_assembly, origin xyz=0.0020000000000000313 -5.598548939047626e-18 0.0400000000000001 rpy=5.551115123125779e-16 4.440892098500626e-16 6.550315845288408e-15, axis -3.2751579226442118e-15 -0.9999999999999977 4.440892098500626e-16, limit lower=-0.2617993877991494 upper=1.8675022996339325 effort=100 velocity=100
- added joint right_pinky_abd: type revolute, parent right_carpals, child right_pinky_ap, origin xyz=0.035641716045904354 0.0006891586859576128 0.06205424192069395 rpy=-1.529473573814961 1.2028622114983025 -2.9119895363116646, axis 9.71445146547012e-16 1.6653345369377348e-16 0.9999999999999984, limit lower=-0.5235987755982988 upper=0.5235987755982988 effort=100 velocity=100
- added joint right_pinky_mcp: type revolute, parent right_pinky_ap, child right_pinky_pp, origin xyz=-0.017750000000000075 -4.698582746252626e-17 -0.0010000000000000768 rpy=0.0 -1.5707963267948908 0.0, axis 6.439293542825908e-15 -1.0000000000000049 6.661338147750939e-16, limit lower=-0.4363323129985824 upper=1.7453292519943295 effort=100 velocity=100
- added joint right_pinky_pip: type revolute, parent right_pinky_pp, child right_pinky_fingertip_assembly, origin xyz=0.000999999999999998 3.208202345938654e-17 0.030999999999999632 rpy=1.1102230246251565e-16 0.0 6.217248937900863e-15, axis -2.609024107869118e-15 -0.9999999999999968 3.885780586188048e-16, limit lower=-0.2617993877991494 upper=1.8675022996339325 effort=100 velocity=100
- added joint right_ring_abd: type revolute, parent right_carpals, child right_ring_ap, origin xyz=0.015307722147416544 -0.003218364665125601 0.07130479703009855 rpy=-1.5707963267948946 1.4250613342533707 -3.054326190990075, axis 8.881784197001252e-16 -5.551115123125783e-17 0.9999999999999994, limit lower=-0.47123889803846897 upper=0.47123889803846897 effort=100 velocity=100
- added joint right_ring_mcp: type revolute, parent right_ring_ap, child right_ring_pp, origin xyz=-0.01986696794290542 3.8657355141463114e-17 -0.00099999999999545 rpy=0.0 -1.5707963267948908 0.0, axis 5.9396931817445875e-15 -1.0000000000000042 1.1102230246251565e-16, limit lower=-0.4363323129985824 upper=1.7453292519943295 effort=100 velocity=100
- added joint right_ring_pip: type revolute, parent right_ring_pp, child right_ring_fingertip_assembly, origin xyz=0.0019999999999998678 1.5882195667426256e-18 0.040000000000000126 rpy=2.2204460492503052e-16 0.0 6.217248937900862e-15, axis -2.942091015256665e-15 -0.999999999999996 2.220446049250313e-16, limit lower=-0.2617993877991494 upper=1.8675022996339325 effort=100 velocity=100
- added joint right_thumb_abd: type revolute, parent right_thumb_tp, child right_thumb_ap, origin xyz=-0.007999999999728488 -1.8648424965940806e-17 -0.003850000000000026 rpy=-1.221730476396032 -1.9984014443252818e-15 -2.3314683517128287e-15, axis -1.4988010832439613e-15 0.3420201433256641 0.9396926207859044, limit lower=-0.3141592653589793 upper=0.9599310885968813 effort=100 velocity=100
- added joint right_thumb_cmc: type revolute, parent right_carpals, child right_thumb_tp, origin xyz=-0.028398719136200776 0.010997180928709077 0.03058953349163134 rpy=0.6614951404674763 0.3860568562160207 -1.4328677049607634, axis -7.771561172376096e-16 5.412337245047638e-16 -0.9999999999999931, limit lower=-0.7853981633974483 upper=0.5759586531581288 effort=100 velocity=100
- added joint right_thumb_dip: type revolute, parent right_thumb_pp, child right_thumb_dp, origin xyz=0.0009999999999999985 1.1880660448999647e-16 0.03200000000000021 rpy=0.0 0.0 -3.830269434956779e-15, axis 4.718447854656915e-16 -0.9999999999999946 3.164135620181696e-15, limit lower=-0.2617993877991494 upper=1.8675022996339325 effort=100 velocity=100
- added joint right_thumb_mcp: type revolute, parent right_thumb_ap, child right_thumb_pp, origin xyz=-0.027999999999999976 4.673366946417151e-18 1.305542026140606e-16 rpy=-3.1415926535897927 1.5707963267948921 0.0, axis -3.1363800445660672e-15 -1.0000000000000027 2.942091015256665e-15, limit lower=-0.4363323129985824 upper=1.7453292519943295 effort=100 velocity=100
- added joint right_tower_fixed: type fixed, parent right_forearm, child right_tower, origin xyz=-0.010000000000000018 0.05230000000000584 -2.0816681711721685e-17 rpy=-1.5707963267948966 1.570796326794894 0.0
- added joint right_wrist: type revolute, parent right_tower, child right_carpals, origin xyz=5.551115123125783e-17 2.3418766925686896e-17 0.04000000000000006 rpy=0.0 0.0 -1.5707963267948992, axis -0.9999999999999963 -1.1270242357758872e-16 5.94450127715256e-17, limit lower=-1.1344640137963142 upper=0.6108652381980153 effort=100 velocity=100

Commit message: Derive v2 inertial properties from the printed parts, skins and servos
The Fusion-exported URDF inertials were wrong in three ways: tensors were in
kg*cm^2 (1e4 too large), the forearm (7.42 kg) and fingertips (~5x) still had
Fusion's default Steel density, and every <inertial> origin sat at the part
frame origin (on the joint axis) with the tensor taken about that point rather
than the centre of mass. The MJCF instead derived mass from the visual meshes
at 1000 kg/m^3, which MuJoCo's legacy mesh inertia overcounts for non-convex
parts. The two models disagreed.

utils/compute_inertials.py now writes both from one source, per link as a sum
of uniform solids:
  - printed PLA parts: masses from slicing orcahand_hardware's Prints-1100.3mf
    with its own settings (PLA+ 1.25 g/cm^3, 15% gyroid), support excluded;
    geometry from the hardware STLs, which share this repo's part frames
  - cast skins: STL volume at an assumed 1100 kg/m^3
  - servos (models from orca_core MOTOR_MODELS, masses from retailer specs):
    16 HLS3915 (35.8 g) spread over the forearm envelope, one HLS3930 (70.5 g)
    over the tower
The COM becomes the URDF <inertial> origin / MJCF <inertial pos>, with the
tensor about it; the MJCF <inertial> overrides the geom-derived values.
mirror_left_from_right.py mirrors MJCF fullinertia (ixy, ixz negated).

Hand mass 967.9 g (was 8.01 kg URDF / 1.76 kg MJCF). Not included: spools,
hulls, fans, electronics, cables, bearings, screws. URDF and MJCF now agree
exactly on every link, and left == mirror(right).

Co-Authored-By: Claude Opus 5.5 <noreply@anthropic.com>

File: v2/models/urdf/orcahand_left.urdf (robot description, URDF)
Before this commit: robot orcahand_left, 19 links, 18 joints
Links:
- link left_carpals: mass 0.13538810897856451 -> 0.0706614
- link left_forearm: mass 7.422534035794272 -> 0.6594
- link left_index_ap: mass 0.004590288233037025 -> 0.00349
- link left_index_fingertip_assembly: mass 0.04675178908397048 -> 0.00807609
- link left_index_pp: mass 0.011373207304546197 -> 0.00906149
- link left_middle_ap: mass 0.004923565158859135 -> 0.00371
- link left_middle_fingertip_assembly: mass 0.04673701376980013 -> 0.008357
- link left_middle_pp: mass 0.012733573971304512 -> 0.010081
- link left_pinky_ap: mass 0.004135862855401387 -> 0.00307
- link left_pinky_fingertip_assembly: mass 0.033190557637887204 -> 0.00630374
- link left_pinky_pp: mass 0.008117379921259958 -> 0.00658097
- link left_ring_ap: mass 0.004923565158859135 -> 0.00371
- link left_ring_fingertip_assembly: mass 0.04673701376980013 -> 0.008357
- link left_ring_pp: mass 0.012733573971304512 -> 0.010081
- link left_thumb_ap: mass 0.007004136465100992 -> 0.00507
- link left_thumb_dp: mass 0.00815768733004441 -> 0.00617055
- link left_thumb_pp: mass 0.010490827160908196 -> 0.00805314
- link left_thumb_tp: mass 0.00797873207561227 -> 0.00554
- link left_tower: mass 0.18565193224536478 -> 0.1321

File: v2/models/urdf/orcahand_right.urdf (robot description, URDF)
Before this commit: robot orcahand_right, 19 links, 18 joints
Links:
- link right_carpals: mass 0.13538810897856451 -> 0.0706614
- link right_forearm: mass 7.422534035794272 -> 0.6594
- link right_index_ap: mass 0.004590288233037025 -> 0.00349
- link right_index_fingertip_assembly: mass 0.04675178908397048 -> 0.00807609
- link right_index_pp: mass 0.011373207304546197 -> 0.00906149
- link right_middle_ap: mass 0.004923565158859135 -> 0.00371
- link right_middle_fingertip_assembly: mass 0.04673701376980013 -> 0.008357
- link right_middle_pp: mass 0.012733573971304512 -> 0.010081
- link right_pinky_ap: mass 0.004135862855401387 -> 0.00307
- link right_pinky_fingertip_assembly: mass 0.033190557637887204 -> 0.00630374
- link right_pinky_pp: mass 0.008117379921259958 -> 0.00658097
- link right_ring_ap: mass 0.004923565158859135 -> 0.00371
- link right_ring_fingertip_assembly: mass 0.04673701376980013 -> 0.008357
- link right_ring_pp: mass 0.012733573971304512 -> 0.010081
- link right_thumb_ap: mass 0.007004136465100992 -> 0.00507
- link right_thumb_dp: mass 0.00815768733004441 -> 0.00617055
- link right_thumb_pp: mass 0.010490827160908196 -> 0.00805314
- link right_thumb_tp: mass 0.00797873207561227 -> 0.00554
- link right_tower: mass 0.18565193224536478 -> 0.1321
