Commit message: Rebuild v2 palm and finger collision hulls to stop palm self-collisions
In URDF-based simulators with self-collision enabled (only parent-child pairs
filtered, e.g. Isaac/PhysX), the palm hulls intersected non-adjacent links
across their normal range of motion, which made GPU PhysX unstable:
  - the distal palm hull bridged the valleys between the knuckle housings and
    the clevis slot each knuckle sits in: proximal phalanges went up to 3.6 mm
    into it during abduction;
  - the proximal palm hull filled the thumb pocket: thumb_ap went up to 7.5 mm
    into it (1.8 mm already at rest).
This repo's palm mesh is also an older revision lying up to 4 mm outside the
printed palm.

make_collision_hulls.py now builds finger, thumb and palm hulls from the
printed parts in orcahand_hardware (orca_v2/base, same part frames; pass
--hardware if not checked out next to this repo) and cuts with arbitrary
planes:
  - palm: 21 pieces along its real features: dorsal/palmar wall of each
    knuckle slot, cuts at the valleys between knuckles, the ring/pinky step,
    and the thumb pocket split into floor, rim, wall and heel;
  - each finger's proximal phalanx bone split at its neck (z = 9 mm).
The tower keeps its filled envelope hulls; visual meshes are unchanged.

Checked over abduction x MCP (fingers) and CMC x abduction (thumb) against
the printed parts: no hull overlap where the real parts are apart (index: 6
poses <= 0.25 mm at its limit corner, where the real index touches too); at
rest every non-adjacent pair has >= 2.5 mm. Where the real parts touch (index
and thumb limit corners) the hulls overlap 0.3-0.4 mm more. Finger-on-finger
contact when one finger abducts fully into a straight neighbour is real
(printed parts overlap ~5 mm) and unchanged.

53 collision geoms per hand (was 31). MuJoCo: masses unchanged, no
self-contacts at rest or when closing, step time 1.14x v1 (0.94-0.97x
previous). mirror_left_from_right.py now removes left collision hulls whose
right counterpart is gone, and --check reports them.

Co-Authored-By: Claude Opus 5.5 <noreply@anthropic.com>

File: v2/models/urdf/orcahand_left.urdf (robot description, URDF)
Before this commit: robot orcahand_left, 19 links, 18 joints
Links:
- link left_carpals: geometry collision mesh filename=package://orcahand_description/v2/models/assets/left/collis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 scale=0.001 0.001 0.001; collision mesh filename=package://orcahand_description/v2/models/assets/left/collis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 scale=0.001 0.001 0.001
- link left_index_pp: geometry collision mesh filename=package://orcahand_description/v2/models/assets/left/collis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 scale=0.001 0.001 0.001; collision mesh filename=package://orcahand_description/v2/models/assets/left/collis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 scale=0.001 0.001 0.001
- link left_middle_pp: geometry collision mesh filename=package://orcahand_description/v2/models/assets/left/collis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 scale=0.001 0.001 0.001; collision mesh filename=package://orcahand_description/v2/models/assets/left/collis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 scale=0.001 0.001 0.001
- link left_pinky_pp: geometry collision mesh filename=package://orcahand_description/v2/models/assets/left/collis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 scale=0.001 0.001 0.001; collision mesh filename=package://orcahand_description/v2/models/assets/left/collis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 scale=0.001 0.001 0.001
- link left_ring_pp: geometry collision mesh filename=package://orcahand_description/v2/models/assets/left/collis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 scale=0.001 0.001 0.001; collision mesh filename=package://orcahand_description/v2/models/assets/left/collis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 scale=0.001 0.001 0.001

File: v2/models/urdf/orcahand_right.urdf (robot description, URDF)
Before this commit: robot orcahand_right, 19 links, 18 joints
Links:
- link right_carpals: geometry collision mesh filename=package://orcahand_description/v2/models/assets/right/colli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 scale=0.001 0.001 0.001; collision mesh filename=package://orcahand_description/v2/models/assets/right/colli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 scale=0.001 0.001 0.001
- link right_index_pp: geometry collision mesh filename=package://orcahand_description/v2/models/assets/right/colli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 scale=0.001 0.001 0.001; collision mesh filename=package://orcahand_description/v2/models/assets/right/colli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 scale=0.001 0.001 0.001
- link right_middle_pp: geometry collision mesh filename=package://orcahand_description/v2/models/assets/right/colli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 scale=0.001 0.001 0.001; collision mesh filename=package://orcahand_description/v2/models/assets/right/colli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 scale=0.001 0.001 0.001
- link right_pinky_pp: geometry collision mesh filename=package://orcahand_description/v2/models/assets/right/colli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 scale=0.001 0.001 0.001; collision mesh filename=package://orcahand_description/v2/models/assets/right/colli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 scale=0.001 0.001 0.001
- link right_ring_pp: geometry collision mesh filename=package://orcahand_description/v2/models/assets/right/colli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 scale=0.001 0.001 0.001; collision mesh filename=package://orcahand_description/v2/models/assets/right/colli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 scale=0.001 0.001 0.001
